File: Twilight_Adapter.kicad_pcb (KiCad board)
At the start: 2 copper layers, 100 x 40 mm, 24 parts, among them J1 Input_Jack, J2 Output_Jack, J3 PINHD_1x2_Female, J4 PINHD_1x2_Female, J5 Barrel_Jack_Switch, J6 PINHD_2x5_Male, J7 PINHD_2x5_Male, J8 PINHD_1x2_Female, SW1 DPDT, SW2 SW_DIP_x01, SW3 SW_DIP_x01

Commit message: Fix R1 footprint reference on PCB
The R1 resistor footprint had its Reference field set to "10kΩ"
(its value) instead of "R1", which crashed KiBot's BOM generation
and blocked the whole CI run before any output could be produced.
Parts:
- renumbered 10kΩ to R1
Changed lines of the file:
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@@
 		(at 137.5 98)
 		(tags "Resistor")
-		(property "Reference" "10kΩ"
+		(property "Reference" "R1"
 			(at 0 0 0)
 			(unlocked yes)
